Commit message: updated code

File: catkin_ws/src/my_robot/urdf/my_robot.xacro (robot description, xacro)
@@ -141,10 +141,10 @@
     </collision>
   </link>
-  <joint type="fixed" name="camera_joint">
+  <joint name="camera_joint" type="fixed">
     <origin xyz="0.2 0 0" rpy="0 0 0"/>
+    <parent link="chassis"/>
     <child link="camera"/>
-    <parent link="chassis"/>
-    <axis xyz="0 1 0" rpy="0 0 0"/>
-   </joint>
+    <!--axis xyz="0 1 0" rpy="0 0 0"/-->
+  </joint>
   <link name="hokuyo">
     <inertial>
@@ -170,4 +170,12 @@
     </collision>
   </link>
+<link name="camera_link_optical">
+  </link>
+  <joint name="camera_optical_joint" type="fixed">
+    <origin xyz="0 0 0" rpy="-1.5707 0 -1.5707"/>
+    <parent link="camera"/>
+    <child link="camera_link_optical"/>
+    <!--axis xyz="0 1 0" rpy="0 0 0"/-->
+  </joint>
   <joint type="fixed" name="hokuyo_joint">
     <origin xyz="0.15 0 0.1" rpy="0 0 0"/>
@@ -188,3 +196,6 @@
  <material>Gazebo/Yellow</material>
  </gazebo>
+ <gazebo reference="camera_link_optical">
+ <material>Gazebo/Blue</material>
+ </gazebo>
 </robot>

Commit message: updated src same as submitted proj

File: catkin_ws/src/my_robot/urdf/my_robot.xacro (robot description, xacro)
@@ -170,18 +170,17 @@
     </collision>
   </link>
-<link name="camera_link_optical">
-  </link>
+ <joint type="fixed" name="hokuyo_joint">
+    <origin xyz="0.15 0 0.1" rpy="0 0 0"/>
+    <child link="hokuyo"/>
+    <parent link="chassis"/>
+    <axis xyz="0 1 0" rpy="0 0 0"/>
+   </joint>
   <joint name="camera_optical_joint" type="fixed">
     <origin xyz="0 0 0" rpy="-1.5707 0 -1.5707"/>
     <parent link="camera"/>
     <child link="camera_link_optical"/>
-    <!--axis xyz="0 1 0" rpy="0 0 0"/-->
-  </joint>
-  <joint type="fixed" name="hokuyo_joint">
-    <origin xyz="0.15 0 0.1" rpy="0 0 0"/>
-    <child link="hokuyo"/>
-    <parent link="chassis"/>
-    <axis xyz="0 1 0" rpy="0 0 0"/>
-   </joint>
+  </joint>
+<link name="camera_link_optical">
+  </link>
  <gazebo reference="left_wheel">
  <material>Gazebo/Black</material>
